File: latest/Presentation/boards/pedalboard-soundcard.kicad_pcb (KiCad board)
At the start: 2 copper layers, 65 x 56 mm, 83 parts, among them J1 RPi_GPIO, J2 Conn_02x03_Odd_Even, J3 Conn_02x03_Odd_Even, J4 Audio_Jack, J5 Audio_Jack, U1 AT24CS01-STUM, U2 NCP163, U3 NCP163, U4 PCM1863DBT, U5 NCP163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

Commit message: Deploying to main from @ pedalboard/pedalboard-soundcard@5062527d60d1d7cefc9884fb6fbaf3b1f6e79b11 🚀
Parts:
- added T1: Tab, PCM_kikit:Tab, F.Cu at (100.0, 109.0)
- added T2: Tab, PCM_kikit:Tab, F.Cu at (48.0, 65.0)
- added T3: Tab, PCM_kikit:Tab, F.Cu at (100.0, 52.0)
- added T4: Tab, PCM_kikit:Tab, F.Cu at (114.0, 65.0)
Changed lines of the file:
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@@
     (pad_to_mask_clearance 0)
     (aux_axis_origin 48.5 108.5)
+    (grid_origin 48.5 108.5)
     (pcbplotparams
       (layerselection 0x0000030_80000001)
@@
     )
   )
+  (footprint "PCM_kikit:Tab" (layer "F.Cu")
+    (at 114 65 180)
+    (descr "A symbol representing annotation for tab placement")
+    (property "Sheetfile" "pedalboard-soundcard.kicad_sch")
+    (property "Sheetname" "")
+    (property "exclude_from_bom" "")
+    (property "ki_description" "KiKit tab annotations")
+    (property "ki_keywords" "KiKit")
+    (attr exclude_from_pos_files exclude_from_bom)
+    (fp_text reference "T4" (at 0 -2) (layer "F.SilkS") hide
+        (effects (font (size 1 1) (thickness 0.15)))
+    )
+    (fp_text value "Tab" (at -2.75 -1) (layer "Dwgs.User")
+        (effects (font (size 1.2 1.2) (thickness 0.2)))
+    )
+    (fp_text user "KIKIT: width: 5mm" (at -5.5 0 90) (layer "Dwgs.User")
+        (effects (font (size 1 1) (thickness 0.15)))
+    )
+    (fp_line (start 0.25 0) (end -2.75 0)
+      (stroke (width 0.3) (type solid)) (layer "Dwgs.User"))
+    (fp_line (start 0.25 0) (end -0.75 -1)
+      (stroke (width 0.3) (type solid)) (layer "Dwgs.User"))
+    (fp_line (start 0.25 0) (end -0.75 1)
+      (stroke (width 0.3) (type solid)) (layer "Dwgs.User"))
+    (fp_line (start 0.25 1) (end 0.25 -1)
+      (stroke (width 0.3) (type solid)) (layer "Dwgs.User"))
+  )
   (footprint "Resistor_SMD:R_0805_2012Metric" (layer "F.Cu")
     (at 84.15 73.88 90)
@@
     )
   )
+  (footprint "PCM_kikit:Tab" (layer "F.Cu")
+    (at 100 109 90)
+    (descr "A symbol representing annotation for tab placement")
+    (property "Sheetfile" "pedalboard-soundcard.kicad_sch")
+    (property "Sheetname" "")
+    (property "exclude_from_bom" "")
+    (property "ki_description" "KiKit tab annotations")
+    (property "ki_keywords" "KiKit")
+    (attr exclude_from_pos_files exclude_from_bom)
+    (fp_text reference "T1" (at 0 -2 90) (layer "F.SilkS") hide
+        (effects (font (size 1 1) (thickness 0.15)))
+    )
+    (fp_text value "Tab" (at -2.75 -1 90) (layer "Dwgs.User")
+        (effects (font (size 1.2 1.2) (thickness 0.2)))
+    )
+    (fp_text user "KIKIT: width: 5mm" (at -5.5 0) (layer "Dwgs.User")
+        (effects (font (size 1 1) (thickness 0.15)))
+    )
+    (fp_line (start 0.25 0) (end -2.75 0)
+      (stroke (width 0.3) (type solid)) (layer "Dwgs.User"))
+    (fp_line (start 0.25 0) (end -0.75 -1)
+      (stroke (width 0.3) (type solid)) (layer "Dwgs.User"))
+    (fp_line (start 0.25 0) (end -0.75 1)
+      (stroke (width 0.3) (type solid)) (layer "Dwgs.User"))
+    (fp_line (start 0.25 1) (end 0.25 -1)
+      (stroke (width 0.3) (type solid)) (layer "Dwgs.User"))
+  )
   (footprint "LED_SMD:LED_0805_2012Metric" (layer "F.Cu")
     (at 58.505 79.75)
@@
       (solder_mask_margin 0.375) (clearance 0.375))
   )
+  (footprint "PCM_kikit:Tab" (layer "F.Cu")
+    (at 100 52 -90)
+    (descr "A symbol representing annotation for tab placement")
+    (property "Sheetfile" "pedalboard-soundcard.kicad_sch")
+    (property "Sheetname" "")
+    (property "exclude_from_bom" "")
+    (property "ki_description" "KiKit tab annotations")
+    (property "ki_keywords" "KiKit")
+    (attr exclude_from_pos_files exclude_from_bom)
+    (fp_text reference "T3" (at 0 -2 90) (layer "F.SilkS") hide
+        (effects (font (size 1 1) (thickness 0.15)))
+    )
+    (fp_text value "Tab" (at -2.75 -1 90) (layer "Dwgs.User")
+        (effects (font (size 1.2 1.2) (thickness 0.2)))
+    )
+    (fp_text user "KIKIT: width: 5mm" (at -5.5 0) (layer "Dwgs.User")
+        (effects (font (size 1 1) (thickness 0.15)))
+    )
+    (fp_line (start 0.25 0) (end -2.75 0)
+      (stroke (width 0.3) (type solid)) (layer "Dwgs.User"))
+    (fp_line (start 0.25 0) (end -0.75 -1)
+      (stroke (width 0.3) (type solid)) (layer "Dwgs.User"))
+    (fp_line (start 0.25 0) (end -0.75 1)
+      (stroke (width 0.3) (type solid)) (layer "Dwgs.User"))
+    (fp_line (start 0.25 1) (end 0.25 -1)
+      (stroke (width 0.3) (type solid)) (layer "Dwgs.User"))
+  )
   (footprint "Resistor_SMD:R_0805_2012Metric" (layer "F.Cu")
     (at 104.44 90.0775 90)
@@
     )
   )
+  (footprint "PCM_kikit:Tab" (layer "F.Cu")
+    (at 48 65)
+    (descr "A symbol representing annotation for tab placement")
+    (property "Sheetfile" "pedalboard-soundcard.kicad_sch")
+    (property "Sheetname" "")
+    (property "exclude_from_bom" "")
+    (property "ki_description" "KiKit tab annotations")
+    (property "ki_keywords" "KiKit")
+    (attr exclude_from_pos_files exclude_from_bom)
+    (fp_text reference "T2" (at 0 -2) (layer "F.SilkS") hide
+        (effects (font (size 1 1) (thickness 0.15)))
+    )
+    (fp_text value "Tab" (at -2.75 -1) (layer "Dwgs.User")
+        (effects (font (size 1.2 1.2) (thickness 0.2)))
+    )
+    (fp_text user "KIKIT: width: 5mm" (at -5.5 0 90) (layer "Dwgs.User")
+        (effects (font (size 1 1) (thickness 0.15)))
+    )
+    (fp_line (start 0.25 0) (end -2.75 0)
+      (stroke (width 0.3) (type solid)) (layer "Dwgs.User"))
+    (fp_line (start 0.25 0) (end -0.75 -1)
+      (stroke (width 0.3) (type solid)) (layer "Dwgs.User"))
+    (fp_line (start 0.25 0) (end -0.75 1)
+      (stroke (width 0.3) (type solid)) (layer "Dwgs.User"))
+    (fp_line (start 0.25 1) (end 0.25 -1)
+      (stroke (width 0.3) (type solid)) (layer "Dwgs.User"))
+  )
   (footprint "Resistor_SMD:R_0805_2012Metric" (layer "F.Cu")
