File: latest/Presentation/boards/pedalboard-soundcard.kicad_pcb (KiCad board)
At the start: 2 copper layers, 65 x 56 mm, 87 parts, among them J1 RPi_GPIO, J2 Conn_02x03_Odd_Even, J3 Conn_02x03_Odd_Even, J4 Audio_Jack, J5 Audio_Jack, T1 Tab, T2 Tab, T3 Tab, T4 Tab, U1 AT24CS01-STUM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

Commit message: Deploying to main from @ pedalboard/pedalboard-soundcard@cb641f7770a1cd062746c3691cf60e673af2823d 🚀
Parts:
- added JP1: SJP, Jumper:SolderJumper-2_P1.3mm_Open_RoundedPad1.0x1.5mm, F.Cu at (103.0, 100.7)
Connections:
- C21 pad 2: GND -> Net-(JP1-B)
- C22 pad 2: GND -> Net-(JP1-B)
- C25 pad 2: GND -> Net-(JP1-B)
- C26 pad 2: GND -> Net-(JP1-B)
Routing:
- net Net-(JP1-B): track 0.00 -> 6.39 mm, vias 0 -> 2
- net GND: track 61.1 -> 59.3 mm, vias 34 -> 31

Commit message: Deploying to main from @ pedalboard/pedalboard-soundcard@c8ff8143bd6d3519a289d2009de94ac11b01fc0e 🚀
Parts:
- added JP2: SJP, Jumper:SolderJumper-2_P1.3mm_Open_RoundedPad1.0x1.5mm, F.Cu at (104.1, 83.7)
- moved JP1 1.30 mm to (104.3, 100.7), turned to 180 degrees
Connections:
- C25 pad 2: Net-(JP1-B) -> Net-(JP2-B)
- C26 pad 2: Net-(JP1-B) -> Net-(JP2-B)
Routing:
- net Net-(JP2-B): track 0.00 -> 4.03 mm
- net Net-(JP1-B): track 6.39 -> 4.04 mm, vias 2 -> 0
- net GND: track 59.3 -> 60.1 mm, vias 31 -> 34
